File: eagle/PwrRelBr/brd-gates-low.sch (EAGLE design)
At the start: 16 parts

Commit message: further brd optimization
Parts:
- added RG1_A1, RG_1B1: (no value), rcl:R-EU_0207/10
Connections:
- net N$3: now also RG1_A1.1
- net N$4: now also RG_1B1.1
- net N$5: now also RG1_A1.2
- net N$6: now also RG_1B1.2
Changed lines of the file:
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@@
 <setting verticaltext="up"/>
 </settings>
-<grid distance="0.1" unitdist="inch" unit="inch" style="dots" multiple="1" display="yes" altdistance="0.01" altunitdist="inch" altunit="inch"/>
+<grid distance="0.1" unitdist="inch" unit="inch" style="lines" multiple="1" display="no" altdistance="0.01" altunitdist="inch" altunit="inch"/>
 <layers>
 <layer number="1" name="Top" color="4" fill="1" visible="no" active="no"/>
@@
 <part name="R1A" library="rcl" deviceset="R-EU_" device="0207/10"/>
 <part name="R1B" library="rcl" deviceset="R-EU_" device="0207/10"/>
+<part name="RG1_A1" library="rcl" deviceset="R-EU_" device="0207/10"/>
+<part name="RG_1B1" library="rcl" deviceset="R-EU_" device="0207/10"/>
 </parts>
 <sheets>
@@
 <instance part="R1A" gate="G$1" x="86.36" y="45.72" rot="R90"/>
 <instance part="R1B" gate="G$1" x="101.6" y="43.18" rot="R90"/>
+<instance part="RG1_A1" gate="G$1" x="68.58" y="66.04"/>
+<instance part="RG_1B1" gate="G$1" x="68.58" y="50.8"/>
 </instances>
 <busses>
@@
 <pinref part="RG1_A" gate="G$1" pin="1"/>
 <wire x1="55.88" y1="60.96" x2="63.5" y2="60.96" width="0.1524" layer="91"/>
+<pinref part="RG1_A1" gate="G$1" pin="1"/>
+<wire x1="63.5" y1="66.04" x2="63.5" y2="60.96" width="0.1524" layer="91"/>
+<junction x="63.5" y="60.96"/>
 </segment>
 </net>
@@
 <pinref part="RG_1B" gate="G$1" pin="1"/>
 <wire x1="55.88" y1="55.88" x2="63.5" y2="55.88" width="0.1524" layer="91"/>
+<pinref part="RG_1B1" gate="G$1" pin="1"/>
+<wire x1="63.5" y1="50.8" x2="63.5" y2="55.88" width="0.1524" layer="91"/>
+<junction x="63.5" y="55.88"/>
 </segment>
 </net>
@@
 <wire x1="86.36" y1="50.8" x2="86.36" y2="60.96" width="0.1524" layer="91"/>
 <junction x="86.36" y="60.96"/>
+<pinref part="RG1_A1" gate="G$1" pin="2"/>
+<wire x1="73.66" y1="60.96" x2="73.66" y2="66.04" width="0.1524" layer="91"/>
+<junction x="73.66" y="60.96"/>
 </segment>
 </net>
@@
 <wire x1="101.6" y1="48.26" x2="101.6" y2="55.88" width="0.1524" layer="91"/>
 <junction x="101.6" y="55.88"/>
+<pinref part="RG_1B1" gate="G$1" pin="2"/>
+<wire x1="73.66" y1="50.8" x2="73.66" y2="55.88" width="0.1524" layer="91"/>
+<junction x="73.66" y="55.88"/>
 </segment>
 </net>
@@
 <segment>
 <pinref part="IC_PWR_PWM" gate="P" pin="GND"/>
-<wire x1="55.88" y1="53.34" x2="71.12" y2="53.34" width="0.1524" layer="91"/>
-<wire x1="71.12" y1="53.34" x2="71.12" y2="33.02" width="0.1524" layer="91"/>
-<wire x1="71.12" y1="33.02" x2="76.2" y2="33.02" width="0.1524" layer="91"/>
+<wire x1="55.88" y1="53.34" x2="58.42" y2="53.34" width="0.1524" layer="91"/>
+<wire x1="58.42" y1="53.34" x2="58.42" y2="33.02" width="0.1524" layer="91"/>
+<wire x1="58.42" y1="33.02" x2="76.2" y2="33.02" width="0.1524" layer="91"/>
 <pinref part="C1" gate="G$1" pin="2"/>
 <wire x1="76.2" y1="33.02" x2="76.2" y2="38.1" width="0.1524" layer="91"/>
@@
 <segment>
 <pinref part="IC_PWR_PWM" gate="P" pin="VS"/>
-<wire x1="73.66" y1="63.5" x2="55.88" y2="63.5" width="0.1524" layer="91"/>
+<wire x1="58.42" y1="63.5" x2="55.88" y2="63.5" width="0.1524" layer="91"/>
 <pinref part="JP_PWR" gate="G$1" pin="1"/>
-<wire x1="71.12" y1="71.12" x2="73.66" y2="71.12" width="0.1524" layer="91"/>
-<wire x1="73.66" y1="71.12" x2="76.2" y2="71.12" width="0.1524" layer="91"/>
+<wire x1="58.42" y1="71.12" x2="71.12" y2="71.12" width="0.1524" layer="91"/>
+<wire x1="71.12" y1="71.12" x2="76.2" y2="71.12" width="0.1524" layer="91"/>
 <wire x1="71.12" y1="86.36" x2="71.12" y2="71.12" width="0.1524" layer="91"/>
 <wire x1="5.08" y1="86.36" x2="22.86" y2="86.36" width="0.1524" layer="91"/>
 <wire x1="22.86" y1="86.36" x2="71.12" y2="86.36" width="0.1524" layer="91"/>
-<wire x1="73.66" y1="63.5" x2="73.66" y2="71.12" width="0.1524" layer="91"/>
-<junction x="73.66" y="71.12"/>
+<wire x1="58.42" y1="63.5" x2="58.42" y2="71.12" width="0.1524" layer="91"/>
 <pinref part="C1" gate="G$1" pin="1"/>
 <wire x1="76.2" y1="45.72" x2="76.2" y2="71.12" width="0.1524" layer="91"/>
@@
 <wire x1="22.86" y1="40.64" x2="22.86" y2="86.36" width="0.1524" layer="91"/>
 <junction x="22.86" y="86.36"/>
-</segment>
-</net>
+<junction x="71.12" y="71.12"/>
+</segment>
+</net>

Commit message: 2nd pair added
Parts:
- removed JP1: (no value), pinhead:PINHD-1X8
- added C2: (no value), rcl:C-EU050-055X075
- added DA2, DB2: BY251, diode:BY251
- added IC_DRV2: IR4427, ir:IR4427
- added JPA2, JPB2, JP_GND2, JP_PWR2: (no value), dbg-misc:PINHD-1X1
- added JPIN1, JPIN2: (no value), pinhead:PINHD-1X2
- added QA2, QB2: IRLZ44Z, dbg-misc:IRLZ44Z
- added RA2, RB2, RGA2, RGB2, RGDA1, RGDB2: (no value), rcl:R-EU_0207/10
- renumbered C3 to CC, DCL1A to DA1, DCL1A1 to DB1, IC_PWR_PWM to IC_DRV1, JP1_OUT_A to JPA1, JP1_OUT_B to JPB1, JP_GND to JP_GND1, JP_PWR to JP_PWR1, Q_PWM to QA1, Q_PWR to QB1, R1A to RA1, R1B to RB1, RG1_A to RGA1, RG1_A1 to RGDA, RG_1B to RGB1, RG_1B1 to RGDB1
Connections:
- new net GND1: C2.2, DA2.A, DB2.A, IC_DRV2.GND, JP_GND2.1, QA2.S, QB2.S, RA2.1, RB2.1
- new net N$10: QB2.G, RB2.2, RGB2.2, RGDB2.2
- new net N$11: DA2.C, JPA2.1, QA2.D
- new net N$12: DB2.C, JPB2.1, QB2.D
- new net N$13: IC_DRV2.INB, JPIN2.1
- new net N$14: IC_DRV2.INA, JPIN2.2
- new net N$7: IC_DRV2.OUTA, RGA2.1, RGDA1.1
- new net N$8: IC_DRV2.OUTB, RGB2.1, RGDB2.1
- new net N$9: QA2.G, RA2.2, RGA2.2, RGDA1.2
- new net VCC1: C2.1, IC_DRV2.VS, JP_PWR2.1
- net N$1: now also JPIN1.2; no longer JP1.8
- net N$2: now also JPIN1.1; no longer JP1.7

Commit message: 4 pairs
Parts:
- added IC_DRV3, IC_DRV4: IR4427, ir:IR4427
- added JPA3, JPA4, JPB3, JPB4, JP_GND3, JP_GND4, JP_PWR3, JP_PWR4: (no value), dbg-misc:PINHD-1X1
- added JPIN3, JPIN4, JPING1: (no value), pinhead:PINHD-1X2
- added QA3, QA4, QB3, QB4: IRLZ44Z, dbg-misc:IRLZ44Z
- added RA3, RA4, RB3, RB4: (no value), rcl:R-EU_0207/10
Connections:
- new net GND2: IC_DRV3.GND, JP_GND3.1, QA3.S, QB3.S, RA3.1, RB3.1
- new net GND3: IC_DRV4.GND, JP_GND4.1, QA4.S, QB4.S, RA4.1, RB4.1
- new net N$16: IC_DRV3.OUTA, QA3.G, RA3.2
- new net N$17: IC_DRV3.OUTB, QB3.G, RB3.2
- new net N$18: IC_DRV4.OUTA, QA4.G, RA4.2
- new net N$19: IC_DRV4.OUTB, QB4.G, RB4.2
- new net N$20: JPA3.1, QA3.D
- new net N$23: JPB3.1, QB3.D
- new net N$24: IC_DRV3.INB, JPIN3.1
- new net N$25: IC_DRV3.INA, JPIN3.2
- new net N$26: JPA4.1, QA4.D
- new net N$27: JPB4.1, QB4.D
- new net N$28: IC_DRV4.INB, JPIN4.1
- new net N$29: IC_DRV4.INA, JPIN4.2
- new net VCC2: IC_DRV3.VS, JP_PWR3.1
- new net VCC3: IC_DRV4.VS, JP_PWR4.1
- net GND: now also JPING1.1
