File: eagle/PwrRelBr/brd-gates-low.brd (EAGLE design)
At the start: 100 x 80 mm, 16 parts

Commit message: placement steps
Parts:
- moved JP_GND 66.5 mm to (20.3, 76.2), turned to 180 degrees
- moved DCL1A 52.1 mm to (8.89, 67.3), turned to 90 degrees
- moved DCL1A1 35.6 mm to (45.7, 69.8), turned to 90 degrees
- moved JP_PWR 31.5 mm to (63.5, 26.7)
- moved JP1_OUT_B 29.6 mm to (45.7, 55.9)
- moved JP1 26.7 mm to (50.8, 5.08), turned to 180 degrees
- moved C1 20.1 mm to (41.9, 17.8), turned to 270 degrees
- moved JP1_OUT_A 19.8 mm to (20.3, 67.3), turned to 180 degrees
- moved C3 11.4 mm to (11.4, 36.8), turned to 180 degrees
- moved Q_PWM 4.02 mm to (24.1, 67.3)
Routing:
- net GND: track 0.00 -> 193.0 mm
- net VCC: track 0.00 -> 77.5 mm
- net N$22: track 0.00 -> 29.2 mm
- net N$5: track 0.00 -> 29.2 mm
- net N$1: track 0.00 -> 20.3 mm
- net N$6: track 0.00 -> 17.8 mm
- net N$2: track 0.00 -> 17.8 mm
- net N$21: track 0.00 -> 16.5 mm
- net N$4: track 0.00 -> 3.81 mm
- net N$3: track 0.00 -> 3.81 mm
Changed lines of the file:
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@@
 </autorouter>
 <elements>
-<element name="C1" library="rcl" package="C050-055X075" value="" x="25.4" y="6.35"/>
-<element name="C3" library="rcl" package="E5-13" value="" x="6.35" y="26.67"/>
-<element name="DCL1A" library="diode" package="DO201-15" value="BY251" x="60.96" y="66.04"/>
-<element name="DCL1A1" library="diode" package="DO201-15" value="BY251" x="10.16" y="69.85"/>
+<element name="C1" library="rcl" package="C050-055X075" value="" x="41.91" y="17.78" rot="R270"/>
+<element name="C3" library="rcl" package="E5-13" value="" x="11.43" y="36.83" rot="R180"/>
+<element name="DCL1A" library="diode" package="DO201-15" value="BY251" x="8.89" y="67.31" rot="R90"/>
+<element name="DCL1A1" library="diode" package="DO201-15" value="BY251" x="45.72" y="69.85" rot="R90"/>
 <element name="IC_PWR_PWM" library="ir" package="DIL08" value="IR4427" x="31.75" y="17.78">
 <attribute name="MPN" value="IR4427" x="31.75" y="17.78" size="1.778" layer="27" display="off"/>
@@
 <attribute name="OC_NEWARK" value="27C6914" x="31.75" y="17.78" size="1.778" layer="27" display="off"/>
 </element>
-<element name="JP1" library="pinhead" package="1X08" value="" x="77.47" y="6.35"/>
-<element name="JP1_OUT_A" library="dbg-misc" package="1X01" value="" x="6.35" y="53.34" rot="R90"/>
-<element name="JP1_OUT_B" library="dbg-misc" package="1X01" value="" x="24.13" y="76.2" rot="R90"/>
-<element name="JP_GND" library="dbg-misc" package="1X01" value="" x="12.7" y="10.16" rot="R90"/>
-<element name="JP_PWR" library="dbg-misc" package="1X01" value="" x="39.37" y="6.35" rot="R90"/>
-<element name="Q_PWM" library="dbg-misc" package="TO220BH" value="IRLZ44Z" x="22.86" y="63.5" rot="R90"/>
+<element name="JP1" library="pinhead" package="1X08" value="" x="50.8" y="5.08" rot="R180"/>
+<element name="JP1_OUT_A" library="dbg-misc" package="1X01" value="" x="20.32" y="67.31" rot="R180"/>
+<element name="JP1_OUT_B" library="dbg-misc" package="1X01" value="" x="45.72" y="55.88" rot="R90"/>
+<element name="JP_GND" library="dbg-misc" package="1X01" value="" x="20.32" y="76.2" rot="R180"/>
+<element name="JP_PWR" library="dbg-misc" package="1X01" value="" x="63.5" y="26.67" rot="R90"/>
+<element name="Q_PWM" library="dbg-misc" package="TO220BH" value="IRLZ44Z" x="24.13" y="67.31" rot="R90"/>
 <element name="Q_PWR" library="dbg-misc" package="TO220BH" value="IRLZ44Z" x="29.21" y="55.88" rot="R90"/>
 <element name="R1A" library="rcl" package="0207/10" value="" x="25.4" y="44.45"/>
@@
 <contactref element="IC_PWR_PWM" pad="7"/>
 <contactref element="RG1_A" pad="1"/>
-<wire x1="30.48" y1="21.59" x2="30.48" y2="25.4" width="0" layer="19" extent="1-1"/>
+<wire x1="30.48" y1="25.4" x2="30.48" y2="21.59" width="0.4064" layer="16"/>
 </signal>
 <signal name="N$4">
 <contactref element="IC_PWR_PWM" pad="5"/>
 <contactref element="RG_1B" pad="1"/>
-<wire x1="35.56" y1="21.59" x2="35.56" y2="25.4" width="0" layer="19" extent="1-1"/>
+<wire x1="35.56" y1="25.4" x2="35.56" y2="21.59" width="0.4064" layer="16"/>
 </signal>
 <signal name="N$5">
@@
 <contactref element="Q_PWM" pad="G"/>
 <contactref element="R1A" pad="2"/>
-<wire x1="30.48" y1="44.45" x2="29.21" y2="60.96" width="0" layer="19" extent="1-1"/>
-<wire x1="30.48" y1="35.56" x2="30.48" y2="44.45" width="0" layer="19" extent="1-1"/>
+<wire x1="30.48" y1="35.56" x2="30.48" y2="44.45" width="0.4064" layer="16"/>
+<wire x1="30.48" y1="44.45" x2="30.48" y2="64.77" width="0.4064" layer="16"/>
 </signal>
 <signal name="N$6">
@@
 <contactref element="Q_PWR" pad="G"/>
 <contactref element="R1B" pad="2"/>
-<wire x1="35.56" y1="39.37" x2="35.56" y2="53.34" width="0" layer="19" extent="1-1"/>
-<wire x1="35.56" y1="35.56" x2="35.56" y2="39.37" width="0" layer="19" extent="1-1"/>
+<wire x1="35.56" y1="39.37" x2="35.56" y2="35.56" width="0.4064" layer="16"/>
+<wire x1="35.56" y1="39.37" x2="35.56" y2="53.34" width="0.4064" layer="16"/>
 </signal>
 <signal name="GND">
@@
 <contactref element="R1A" pad="1"/>
 <contactref element="R1B" pad="1"/>
-<wire x1="35.56" y1="58.42" x2="68.58" y2="66.04" width="0" layer="19" extent="1-1"/>
-<wire x1="29.21" y1="66.04" x2="35.56" y2="58.42" width="0" layer="19" extent="1-1"/>
-<wire x1="17.78" y1="69.85" x2="29.21" y2="66.04" width="0" layer="19" extent="1-1"/>
-<wire x1="20.32" y1="44.45" x2="35.56" y2="58.42" width="0" layer="19" extent="1-1"/>
-<wire x1="25.4" y1="39.37" x2="20.32" y2="44.45" width="0" layer="19" extent="1-1"/>
-<wire x1="8.89" y1="26.67" x2="25.4" y2="39.37" width="0" layer="19" extent="1-1"/>
-<wire x1="12.7" y1="10.16" x2="8.89" y2="26.67" width="0" layer="19" extent="1-1"/>
-<wire x1="27.94" y1="6.35" x2="12.7" y2="10.16" width="0" layer="19" extent="1-1"/>
-<wire x1="33.02" y1="13.97" x2="27.94" y2="6.35" width="0" layer="19" extent="1-1"/>
+<wire x1="41.91" y1="15.24" x2="41.91" y2="17.78" width="0.4064" layer="16"/>
+<wire x1="41.91" y1="17.78" x2="33.02" y2="17.78" width="0.4064" layer="16"/>
+<wire x1="33.02" y1="13.97" x2="33.02" y2="17.78" width="0.4064" layer="16"/>
+<wire x1="33.02" y1="17.78" x2="8.89" y2="17.78" width="0.4064" layer="16"/>
+<wire x1="8.89" y1="36.83" x2="8.89" y2="17.78" width="0.4064" layer="16"/>
+<wire x1="5.08" y1="44.45" x2="5.08" y2="36.83" width="0.4064" layer="16"/>
+<wire x1="5.08" y1="36.83" x2="8.89" y2="36.83" width="0.4064" layer="16"/>
+<wire x1="20.32" y1="44.45" x2="5.08" y2="44.45" width="0.4064" layer="16"/>
+<wire x1="25.4" y1="39.37" x2="20.32" y2="39.37" width="0.4064" layer="16"/>
+<wire x1="20.32" y1="39.37" x2="20.32" y2="44.45" width="0.4064" layer="16"/>
+<wire x1="30.48" y1="69.85" x2="35.56" y2="69.85" width="0.4064" layer="16"/>
+<wire x1="35.56" y1="69.85" x2="35.56" y2="58.42" width="0.4064" layer="16"/>
+<wire x1="45.72" y1="77.47" x2="35.56" y2="77.47" width="0.4064" layer="16"/>
+<wire x1="35.56" y1="77.47" x2="35.56" y2="76.2" width="0.4064" layer="16"/>
+<wire x1="35.56" y1="76.2" x2="35.56" y2="69.85" width="1.016" layer="16"/>
+<wire x1="20.32" y1="76.2" x2="35.56" y2="76.2" width="1.016" layer="16"/>
+<wire x1="8.89" y1="74.93" x2="8.89" y2="76.2" width="0.4064" layer="16"/>
+<wire x1="8.89" y1="76.2" x2="20.32" y2="76.2" width="0.4064" layer="16"/>
+<wire x1="5.08" y1="44.45" x2="5.08" y2="76.2" width="0.4064" layer="16"/>
+<wire x1="5.08" y1="76.2" x2="8.89" y2="76.2" width="0.4064" layer="16"/>
 </signal>
 <signal name="VCC">
@@
 <contactref element="C1" pad="1"/>
 <contactref element="C3" pad="+"/>
-<wire x1="39.37" y1="6.35" x2="33.02" y2="21.59" width="0" layer="19" extent="1-1"/>
-<wire x1="22.86" y1="6.35" x2="39.37" y2="6.35" width="0" layer="19" extent="1-1"/>
-<wire x1="3.81" y1="26.67" x2="22.86" y2="6.35" width="0" layer="19" extent="1-1"/>
+<wire x1="33.02" y1="21.59" x2="33.02" y2="19.05" width="0.4064" layer="16"/>
+<wire x1="33.02" y1="19.05" x2="39.37" y2="19.05" width="0.4064" layer="16"/>
+<wire x1="39.37" y1="19.05" x2="39.37" y2="20.32" width="0.4064" layer="16"/>
+<wire x1="39.37" y1="20.32" x2="41.91" y2="20.32" width="0.4064" layer="16"/>
+<wire x1="41.91" y1="20.32" x2="63.5" y2="20.32" width="0.4064" layer="16"/>
+<wire x1="63.5" y1="20.32" x2="63.5" y2="26.67" width="0.4064" layer="16"/>
+<wire x1="13.97" y1="36.83" x2="13.97" y2="19.05" width="0.4064" layer="16"/>
+<wire x1="13.97" y1="19.05" x2="33.02" y2="19.05" width="0.4064" layer="16"/>
 </signal>
 <signal name="N$22">
@@
 <contactref element="DCL1A" pad="C"/>
 <contactref element="JP1_OUT_A" pad="1"/>
-<wire x1="29.21" y1="63.5" x2="53.34" y2="66.04" width="0" layer="19" extent="1-1"/>
-<wire x1="6.35" y1="53.34" x2="29.21" y2="63.5" width="0" layer="19" extent="1-1"/>
+<wire x1="20.32" y1="67.31" x2="30.48" y2="67.31" width="0.4064" layer="16"/>
+<wire x1="20.32" y1="67.31" x2="20.32" y2="59.69" width="0.4064" layer="16"/>
+<wire x1="20.32" y1="59.69" x2="8.89" y2="59.69" width="0.4064" layer="16"/>
 </signal>
 <signal name="N$21">
@@
 <contactref element="JP1_OUT_B" pad="1"/>
 <contactref element="DCL1A1" pad="C"/>
-<wire x1="2.54" y1="69.85" x2="24.13" y2="76.2" width="0" layer="19" extent="1-1"/>
-<wire x1="35.56" y1="55.88" x2="24.13" y2="76.2" width="0" layer="19" extent="1-1"/>
+<wire x1="45.72" y1="55.88" x2="35.56" y2="55.88" width="0.4064" layer="16"/>
+<wire x1="45.72" y1="62.23" x2="45.72" y2="55.88" width="0.4064" layer="16"/>
 </signal>
 <signal name="N$2">
 <contactref element="JP1" pad="7"/>
 <contactref element="IC_PWR_PWM" pad="4"/>
-<wire x1="35.56" y1="13.97" x2="83.82" y2="6.35" width="0" layer="19" extent="1-1"/>
+<wire x1="35.56" y1="13.97" x2="35.56" y2="11.43" width="0.4064" layer="16"/>
+<wire x1="35.56" y1="11.43" x2="44.45" y2="11.43" width="0.4064" layer="16"/>
+<wire x1="44.45" y1="11.43" x2="44.45" y2="5.08" width="0.4064" layer="16"/>
 </signal>
 <signal name="N$1">
 <contactref element="IC_PWR_PWM" pad="2"/>
 <contactref element="JP1" pad="8"/>
-<wire x1="30.48" y1="13.97" x2="86.36" y2="6.35" width="0" layer="19" extent="1-1"/>
+<wire x1="30.48" y1="13.97" x2="30.48" y2="8.89" width="0.4064" layer="16"/>
+<wire x1="30.48" y1="8.89" x2="41.91" y2="8.89" width="0.4064" layer="16"/>
+<wire x1="41.91" y1="8.89" x2="41.91" y2="5.08" width="0.4064" layer="16"/>
 </signal>
 </signals>

Commit message: further brd optimization
Parts:
- added RG1_A1, RG_1B1: (no value), rcl:0207/10
- moved JP_PWR 56.4 mm to (11.4, 48.3)
- moved C1 26.5 mm to (16.5, 25.4)
- moved C3 24.3 mm to (8.89, 61.0)
- moved JP1_OUT_A 16.6 mm to (19.1, 50.8), turned to 270 degrees
- moved JP1_OUT_B 15.3 mm to (31.8, 49.5)
- moved DCL1A1 15.3 mm to (31.8, 63.5)
- moved RG_1B 11.7 mm to (27.9, 39.4)
- moved JP_GND 11.4 mm to (8.89, 76.2)
- moved R1B 10.9 mm to (20.3, 43.2)
- moved IC_PWR_PWM 10.8 mm to (24.1, 25.4)
- moved DCL1A 10.5 mm to (19.1, 64.8)
- moved RG1_A 9.16 mm to (22.9, 35.6)
- moved Q_PWR 7.62 mm to (21.6, 55.9)
- moved JP1 7.62 mm to (43.2, 5.08)
- moved Q_PWM 7.62 mm to (16.5, 67.3)
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Connections:
- net N$3: now also RG1_A1.1
- net N$4: now also RG_1B1.1
- net N$5: now also RG1_A1.2
- net N$6: now also RG_1B1.2
Routing:
- net GND: track 193.0 -> 179.1 mm
- net N$22: track 29.2 -> 20.3 mm
- net N$2: track 17.8 -> 25.4 mm
- net N$1: track 20.3 -> 27.9 mm
- net VCC: track 77.5 -> 71.1 mm
- net N$21: track 16.5 -> 10.2 mm
- net N$4: track 3.81 -> 8.89 mm
- net N$5: track 29.2 -> 30.5 mm
- net N$3: track 3.81 -> 5.08 mm
- net N$6: track 17.8 -> 16.5 mm

Commit message: 2nd pair added
Parts:
- removed JP1: (no value), pinhead:1X08
- added C2: (no value), rcl:C050-055X075
- added DA2, DB2: BY251, diode:DO201-15
- added IC_DRV2: IR4427, ir:DIL08
- added JPA2, JPB2, JP_GND2, JP_PWR2: (no value), dbg-misc:1X01
- added JPIN1, JPIN2: (no value), pinhead:1X02
- added QA2, QB2: IRLZ44Z, dbg-misc:TO220BH
- added RA2, RB2, RGA2, RGB2, RGDA1, RGDB2: (no value), rcl:0207/10
- renumbered C3 to CC, DCL1A to DA1, DCL1A1 to DB1, IC_PWR_PWM to IC_DRV1, JP1_OUT_A to JPA1, JP1_OUT_B to JPB1, JP_GND to JP_GND1, JP_PWR to JP_PWR1, Q_PWM to QA1, Q_PWR to QB1, R1A to RA1, R1B to RB1, RG1_A to RGA1, RG1_A1 to RGDA, RG_1B to RGB1, RG_1B1 to RGDB1
Connections:
- new net GND1: C2.2, DA2.A, DB2.A, IC_DRV2.3, JP_GND2.1, QA2.S, QB2.S, RA2.1, RB2.1
- new net N$10: QB2.G, RB2.2, RGB2.2, RGDB2.2
- new net N$11: DA2.C, JPA2.1, QA2.D
- new net N$12: DB2.C, JPB2.1, QB2.D
- new net N$13: IC_DRV2.4, JPIN2.1
- new net N$14: IC_DRV2.2, JPIN2.2
- new net N$7: IC_DRV2.7, RGA2.1, RGDA1.1
- new net N$8: IC_DRV2.5, RGB2.1, RGDB2.1
- new net N$9: QA2.G, RA2.2, RGA2.2, RGDA1.2
- new net VCC1: C2.1, IC_DRV2.6, JP_PWR2.1
- net N$1: now also JPIN1.2; no longer JP1.8
- net N$2: now also JPIN1.1; no longer JP1.7
Routing:
- net GND1: track 0.00 -> 109.2 mm
- net VCC1: track 0.00 -> 39.4 mm
- net N$9: track 0.00 -> 30.5 mm
- net N$11: track 0.00 -> 20.3 mm
- net N$1: track 27.9 -> 45.7 mm
- net N$10: track 0.00 -> 16.5 mm
- net N$12: track 0.00 -> 10.2 mm
- net N$8: track 0.00 -> 8.89 mm
- net N$2: track 25.4 -> 33.0 mm
- net N$7: track 0.00 -> 5.08 mm
- net N$15: track 0.00 -> 5.08 mm

Commit message: 4 pairs
Parts:
- added IC_DRV3, IC_DRV4: IR4427, ir:DIL08
- added JPA3, JPA4, JPB3, JPB4, JP_GND3, JP_GND4, JP_PWR3, JP_PWR4: (no value), dbg-misc:1X01
- added JPIN3, JPIN4, JPING1: (no value), pinhead:1X02
- added QA3, QA4, QB3, QB4: IRLZ44Z, dbg-misc:TO220BH
- added RA3, RA4, RB3, RB4: (no value), rcl:0207/10
- moved JPIN2 26.9 mm to (44.5, 12.7)
- moved JPIN1 4.02 mm to (44.5, 8.89)
Connections:
- new net GND2: IC_DRV3.3, JP_GND3.1, QA3.S, QB3.S, RA3.1, RB3.1
- new net GND3: IC_DRV4.3, JP_GND4.1, QA4.S, QB4.S, RA4.1, RB4.1
- new net N$16: IC_DRV3.7, QA3.G, RA3.2
- new net N$17: IC_DRV3.5, QB3.G, RB3.2
- new net N$18: IC_DRV4.7, QA4.G, RA4.2
- new net N$19: IC_DRV4.5, QB4.G, RB4.2
- new net N$20: JPA3.1, QA3.D
- new net N$23: JPB3.1, QB3.D
- new net N$24: IC_DRV3.4, JPIN3.1
- new net N$25: IC_DRV3.2, JPIN3.2
- new net N$26: JPA4.1, QA4.D
- new net N$27: JPB4.1, QB4.D
- new net N$28: IC_DRV4.4, JPIN4.1
- new net N$29: IC_DRV4.2, JPIN4.2
- new net VCC2: IC_DRV3.6, JP_PWR3.1
- new net VCC3: IC_DRV4.6, JP_PWR4.1
- net GND: now also JPING1.1
Routing:
- net GND2: track 0.00 -> 99.1 mm
- net GND3: track 0.00 -> 90.2 mm
- net N$28: track 0.00 -> 46.3 mm
- net N$16: track 0.00 -> 45.7 mm
- net N$18: track 0.00 -> 45.7 mm
- net VCC2: track 0.00 -> 36.8 mm
- net N$29: track 0.00 -> 34.5 mm
- net VCC3: track 0.00 -> 30.5 mm
- net N$19: track 0.00 -> 26.7 mm
- net N$17: track 0.00 -> 26.7 mm
- net N$24: track 0.00 -> 24.4 mm
- net N$25: track 0.00 -> 21.2 mm
- net N$1: track 45.7 -> 31.4 mm
- net N$2: track 33.0 -> 20.5 mm
- net GND: track 179.1 -> 188.8 mm
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